File: hw/stm32_board_2025.kicad_pcb (KiCad board)
At the start: 2 copper layers, 75.1 x 43.7 mm, 44 parts, among them J1 Connector, J2 Connector, J3 Ext. LEDs, Q1 MMBT3904, SW1 SW_Push, SW2 SW_Push, SW3 SW_Push, U1 74HC595, U2 74HC595, U3 D198K, U4 D198K, U5 DS18B20

Commit message: Routed.
Parts:
- moved C4 84.4 mm to (174.0, 117.5), turned to -90 degrees
- moved RV1 83.9 mm to (123.2, 118.7), turned to 90 degrees
- moved R18 82.6 mm to (148.0, 109.9), turned to 180 degrees
- moved C1 81.8 mm to (131.4, 101.0)
- moved R17 80.8 mm to (148.0, 104.8), turned to 180 degrees
- moved R14 80.0 mm to (111.8, 111.8), turned to 180 degrees
- moved R10 79.8 mm to (148.0, 107.3), turned to 180 degrees
- moved R13 79.5 mm to (111.8, 108.0), turned to 180 degrees
- moved R1 78.5 mm to (170.2, 97.8), turned to 180 degrees
- moved R9 78.0 mm to (148.0, 102.2), turned to 180 degrees
- moved R2 77.8 mm to (170.2, 100.3), turned to 180 degrees
- moved R11 77.2 mm to (114.9, 100.3), turned to 90 degrees
- moved R12 76.6 mm to (109.9, 100.3), turned to 90 degrees
- moved R3 74.0 mm to (117.5, 100.3), turned to 90 degrees
- moved R6 73.9 mm to (116.8, 109.9), turned to 180 degrees
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Connections:
- BZ1 pad 1: VDD -> +3.3V
- R1 pad 2: /PA10 -> /PA9
- R2 pad 2: /PA9 -> /PA10
- R20 pad 1: VDD -> +3.3V
- SW1 pad 1: /PA10 -> /PA9
- SW2 pad 1: /PA9 -> /PA10
Routing:
- net +3.3V: track 0.00 -> 150.1 mm, vias 0 -> 6
- net +5V: track 0.00 -> 95.6 mm, vias 0 -> 1
- net /PB1: track 0.00 -> 75.0 mm, vias 0 -> 1
- net /PA0: track 0.00 -> 70.1 mm
- net /PA4: track 0.00 -> 69.4 mm, vias 0 -> 3
- net Net-(D3-DOUT): track 0.00 -> 60.0 mm, vias 0 -> 2
- net /PA9: track 0.00 -> 52.8 mm, vias 0 -> 2
- net /PA5: track 0.00 -> 49.4 mm, vias 0 -> 1
- net /PF0: track 0.00 -> 48.3 mm
- net GND: track 0.00 -> 47.5 mm, vias 0 -> 92
- net /PA10: track 0.00 -> 44.1 mm, vias 0 -> 2
- net /PA7: track 0.00 -> 42.8 mm, vias 0 -> 1
- net Net-(U1-QH'): track 0.00 -> 38.5 mm, vias 0 -> 2
- net Net-(U3-G): track 0.00 -> 37.2 mm, vias 0 -> 2
- net Net-(U3-B): track 0.00 -> 35.7 mm
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- added copper zone on B.Cu, net GND
- added copper zone on F.Cu, net GND

Commit message: Sent to fab.
Parts:
- added G***: LOGO, footprints:MITlogo, F.Cu at (137.8, 105.4)
- added G***: LOGO, footprints:VIKlogo, B.Cu at (121.3, 104.8)
- moved R18 2.54 mm to (170.2, 97.8)
- moved R19 2.54 mm to (170.2, 100.3)
- renumbered C3 to C1, C1 to C2, C2 to C3, D3 to D1, D1 to D3, J2 to J1, J3 to J2, J1 to J3, R12 to R1, R15 to R10, R8 to R11, R16 to R12, R9 to R13, R17 to R14, R10 to R15, R18 to R16, R20 to R17, R2 to R18, R1 to R19, R13 to R2, R21 to R20, R19 to R21, R23 to R22, R22 to R23, R14 to R3, R11 to R5, R5 to R6, R6 to R7, R3 to R8, R7 to R9, U3 to U1, U1 to U2, U4 to U3, U2 to U4
Other:
- board text added: "Buzzer: PA6 (TIM16_CH1) 1wire temp. sensor: PF1 Potentiometer: PA0 (ADC IN0) USART2 TX: PA2 USART2 RX: PA3 Programmer: PA13, PA14"
- board text added: "Display data in: PA7 (SPI1 MOSI) Display clock: PA5 (SPI1 SCK) Display data valid: PA4 (SPI1 nSS) Addressable LEDs: PB1 (TIM3_CH4) Normal LED: PA1"
- board text added: "Rev.A"
- board text added: "SW1: PA9 SW2: PA10 SW3: PF0"
- board text added: "V_IMSC1 tankör 2024/25"
- board text added: "Vesztettem"
