File: hw/stm32_board_2025.kicad_sch (KiCad schematic)
At the start: 44 parts, among them J1 Connector, J2 Connector, J3 Ext. LEDs, Q1 MMBT3904, SW1 SW_Push, SW2 SW_Push, SW3 SW_Push, U1 74HC595, U2 74HC595, U3 D198K, U4 D198K, U5 DS18B20

Commit message: Routed.
Connections:
- net VDD is gone; now on net +3.3V: BZ1.1 (-), R20.1
- net PA10: now also R2.2, SW2.1; no longer R1.2, SW1.1
- net PA9: now also R1.2, SW1.1; no longer R2.2, SW2.1
Changed lines of the file:
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@@
 	)
 	(junction
-		(at 154.94 101.6)
+		(at 31.75 53.34)
 		(diameter 0)
 		(color 0 0 0 0)
 	)
 	(junction
-		(at 31.75 53.34)
+		(at 154.94 101.6)
 		(diameter 0)
 		(color 0 0 0 0)
@@
 		)
 	)
+	(label "PA10"
+		(at 72.39 165.1 180)
+		(effects
+			(font
+				(size 1.27 1.27)
+			)
+			(justify right bottom)
+		)
+	)
 	(label "PF0"
 		(at 152.4 41.91 0)
@@
 		)
 	)
-	(label "PA10"
-		(at 50.8 166.37 180)
-		(effects
-			(font
-				(size 1.27 1.27)
-			)
-			(justify right bottom)
-		)
-	)
 	(label "PA9"
-		(at 72.39 165.1 180)
+		(at 50.8 166.37 180)
 		(effects
 			(font
@@
 	)
 	(symbol
+		(lib_id "power:VCC")
+		(at 154.94 101.6 0)
+		(unit 1)
+		(exclude_from_sim no)
+		(in_bom yes)
+		(on_board yes)
+		(dnp no)
+		(property "Reference" "#PWR021"
+			(at 154.94 105.41 0)
+			(effects
+				(font
+					(size 1.27 1.27)
+				)
+				(hide yes)
+			)
+		)
+		(property "Value" "+3.3V"
+			(at 151.892 97.536 0)
+			(effects
+				(font
+					(size 1.27 1.27)
+				)
+				(justify left)
+			)
+		)
+		(property "Footprint" ""
+			(at 154.94 101.6 0)
+			(effects
+				(font
+					(size 1.27 1.27)
+				)
+				(hide yes)
+			)
+		)
+		(property "Datasheet" ""
+			(at 154.94 101.6 0)
+			(effects
+				(font
+					(size 1.27 1.27)
+				)
+				(hide yes)
+			)
+		)
+		(property "Description" "Power symbol creates a global label with name \"VCC\""
+			(at 154.94 101.6 0)
+			(effects
+				(font
+					(size 1.27 1.27)
+				)
+				(hide yes)
+			)
+		)
+		(pin "1"
+		)
+		(instances
+			(project "stm32_board_2025"
+				(path "/805732fc-2965-45cc-b364-e77e100b39c6"
+					(reference "#PWR021")
+					(unit 1)
+				)
+			)
+		)
+	)
+	(symbol
 		(lib_id "power:GND")
 		(at 110.49 58.42 0)
@@
 					(unit 1)
 				)
-			)
-		)
-	)
-	(symbol
-		(lib_id "power:VDD")
-		(at 154.94 101.6 0)
-		(unit 1)
-		(exclude_from_sim no)
-		(in_bom yes)
-		(on_board yes)
-		(dnp no)
-		(fields_autoplaced yes)
-		(property "Reference" "#PWR021"
-			(at 154.94 105.41 0)
-			(effects
-				(font
-					(size 1.27 1.27)
-				)
-				(hide yes)
-			)
-		)
-		(property "Value" "VDD"
-			(at 154.94 97.79 0)
-			(effects
-				(font
-					(size 1.27 1.27)
-				)
-			)
-		)
-		(property "Footprint" ""
-			(at 154.94 101.6 0)
-			(effects
-				(font
-					(size 1.27 1.27)
-				)
-				(hide yes)
-			)
-		)
-		(property "Datasheet" ""
-			(at 154.94 101.6 0)
-			(effects
-				(font
-					(size 1.27 1.27)
-				)
-				(hide yes)
-			)
-		)
-		(property "Description" ""
-			(at 154.94 101.6 0)
-			(effects
-				(font
-					(size 1.27 1.27)
-				)
-				(hide yes)
-			)
-		)
-		(pin "1"
-		)
-		(instances
-			(project "stm32_board_2025"
-				(path "/805732fc-2965-45cc-b364-e77e100b39c6"
-					(reference "#PWR021")
-					(unit 1)
-				)

Commit message: Sent to fab.
Parts:
- R1: renamed from R12; value 750 -> 1k
- R10: renamed from R15; value 750 -> 1k
- R11: renamed from R8; value 750 -> 1k
- R12: renamed from R16; value 750 -> 1k
- R13: renamed from R9; value 750 -> 1k
- R14: renamed from R17; value 750 -> 1k
- R15: renamed from R10; value 750 -> 1k
- R16: renamed from R18; value 750 -> 1k
- R18: renamed from R2; value 10k -> 1k
- R19: renamed from R1; value 10k -> 1k
- R2: renamed from R13; value 750 -> 1k
- R21: renamed from R19; value 10k -> 1k
- R22: renamed from R23; value 4,7k -> 1k
- R23: renamed from R22; value 750 -> 1k
- R3: renamed from R14; value 750 -> 1k
- R4: value 750 -> 1k
- R5: renamed from R11; value 750 -> 1k
- R6: renamed from R5; value 750 -> 1k
- R7: renamed from R6; value 750 -> 1k
- R8: renamed from R3; value 750 -> 1k
- R9: renamed from R7; value 750 -> 1k
- renumbered C3 to C1, C1 to C2, C2 to C3, D3 to D1, D1 to D3, J2 to J1, J3 to J2, J1 to J3, R20 to R17, R21 to R20, U3 to U1, U1 to U2, U4 to U3, U2 to U4
